File: kicad/analog_input.kicad_sch (KiCad schematic)
At the start: 32 parts, among them U3 LTC2380CMS-24#PBF, U7 THS4561IDGKx

Commit message: bugfix: driver for 4th T, capacitors for input amps
Parts:
- C13, C16: value GCM31CR71C106KA64L -> GCM31CR71C106KA64L
- U3: value LTC2380CMS-24#PBF -> LTC2380CMS-24#PBF
