File: kicad/delta_control.kicad_sch (KiCad schematic)
At the start: 15 parts, among them J14 N2516-6002-RB, J8 L17DAFRA15S, U20 TLP2361(TPL,E, U21 TLP175A, U22 TLP2361(TPL,E

Commit message: bugfix: driver for 4th T, capacitors for input amps
Parts:
- U20, U22: value TLP2361(TPL,E -> TLP2361(TPL,E
