File: kicad/digital_IO.kicad_sch (KiCad schematic)
At the start: 48 parts, among them J6 N2514-6002RB, U10 TLP2361(TPL,E, U11 TLP2361(TPL,E, U12 TLP701AF(F), U13 TLP701AF(F), U14 TLP701AF(F), U15 TLP701AF(F), U16 NL17SZ16DFT2G, U17 TME1215S, U8 NC7WZ17P6X, U9 TLP2361(TPL,E

Commit message: bugfix: driver for 4th T, capacitors for input amps
Parts:
- U10, U11, U9: value TLP2361(TPL,E -> TLP2361(TPL,E
